Commit message: Commenting out collision meshes in URDF
Because rerun displays both meshes, sometimes they collide. Commenting
out for now until this can be fixed on rerun's side.

Also setting the default color to white.

File: lerobot/urdf/so100_follower/so100_follower.urdf (robot description, URDF)
Before this commit: robot so100_follower, 7 links, 6 joints
Links:
- link base: geometry visual mesh filename=assets/Base.stl; visual mesh filename=assets/Base_Motor.stl
- link lower_arm: geometry visual mesh filename=assets/Lower_Arm.stl; visual mesh filename=assets/Lower_Arm_Motor.stl
- link shoulder: geometry visual mesh filename=assets/Rotation_Pitch.stl; visual mesh filename=assets/Rotation_Pitch_Motor.stl
- link upper_arm: geometry visual mesh filename=assets/Upper_Arm.stl; visual mesh filename=assets/Upper_Arm_Motor.stl
- link wrist: geometry visual mesh filename=assets/Wrist_Pitch_Roll.stl; visual mesh filename=assets/Wrist_Pitch_Roll_Motor.stl

File: lerobot/urdf/so101_follower/so101_follower.urdf (robot description, URDF)
Before this commit: robot so101_follower, 7 links, 6 joints
Links:
- link base: geometry visual mesh filename=assets/base_motor_holder_so101_v1.stl; visual mesh filename=assets/base_so101_v2.stl
- link gripper: geometry visual mesh filename=assets/sts3215_03a_v1.stl; visual mesh filename=assets/wrist_roll_follower_so101_v1.stl
- link jaw: geometry visual mesh filename=assets/moving_jaw_so101_v1.stl
- link lower_arm: geometry visual mesh filename=assets/motor_holder_so101_wrist_v1.stl; visual mesh filename=assets/sts3215_03a_v1.stl
- link shoulder: geometry visual mesh filename=assets/motor_holder_so101_base_v1.stl; visual mesh filename=assets/rotation_pitch_so101_v1.stl
- link upper_arm: geometry visual mesh filename=assets/sts3215_03a_v1.stl; visual mesh filename=assets/upper_arm_so101_v1.stl
- link wrist: geometry visual mesh filename=assets/sts3215_03a_no_horn_v1.stl; visual mesh filename=assets/wrist_roll_pitch_so101_v2.stl
